File: boards/LD APD M mount pcb/LD APD M mount.kicad_sch (KiCad schematic)
At the start: 23 parts, among them J3 Conn_01x10, U1 SensL_SiPM

Commit message: made macro system pcb v2
Parts:
- removed APD+, APD-1, GND1, GND2, Laser/pwm, Laser/sup, X+1, X-1, Y+1, Y-1: TestPoint, TestPoint:TestPoint_Pad_2.0x2.0mm, symbol Connector:TestPoint
- removed C1, C2: 1u, Capacitor_SMD:C_0402_1005Metric, symbol Device:C_Small
- removed C3: 0.1u, Capacitor_SMD:C_0402_1005Metric, symbol Device:C_Small
- removed L1: 4.7u, Inductor_SMD:L_0805_2012Metric_Pad1.05x1.20mm_HandSolder, symbol Device:L_Small
- removed R1: 2, Resistor_SMD:R_0402_1005Metric, symbol Device:R_Small_US
- removed R2, R4: 4.7k, Resistor_SMD:R_0402_1005Metric, symbol Device:R_Small_US
- removed R3: 33k, Resistor_SMD:R_0402_1005Metric, symbol Device:R_Small_US
- removed U2: ~, Package_TO_SOT_SMD:SOT-23-6_Handsoldering, symbol 0_kicad_custom_symbols:AP3036
- added J1: Conn_01x10, Connector_PinHeader_2.54mm:PinHeader_1x10_P2.54mm_Vertical, symbol Connector_Generic:Conn_01x10
- U1: footprint footprints:LaserDiode -> 0_kicad_custom_footprints:SensL_SiPM_6mm
Connections:
- net GND: now also U3.13 (GND), U3.18 (GND), U3.3 (GND), U3.8 (GND), J1.10 (Pin_10)
- net at J3.6 (Pin_6), U3.1 (Y+), U3.11 (Y+): now also J1.6 (Pin_6)
- net at U1.3 (Cathode): now also J3.2 (Pin_2), J1.2 (Pin_2); no longer J3.9 (Pin_9)
- net at LD1.3 (C): now also J3.5 (Pin_5), J1.5 (Pin_5)
- net SiPM-: now reaches U1.1 (Anode)
- net SiPM-: now also J3.1 (Pin_1), J1.1 (Pin_1); no longer J3.2 (Pin_2)
- net X-: now reaches U3.15 (X-), U3.5 (X-)
- net X-: now also J3.9 (Pin_9), J1.9 (Pin_9); no longer J3.3 (Pin_3)
- net at U3.16 (X+), U3.6 (X+): now also J3.8 (Pin_8), J1.8 (Pin_8); no longer J3.4 (Pin_4)
- net at U3.10 (Y-), U3.20 (Y-): now also J3.7 (Pin_7), J1.7 (Pin_7); no longer J3.5 (Pin_5)
- net at LD1.1 (A): now also J3.4 (Pin_4), J1.4 (Pin_4)
- now unconnected: U3.12 (NC), U3.14 (NC), U3.17 (NC), U3.19 (NC), U3.2 (NC), U3.4 (NC), U3.7 (NC), U3.9 (NC)
- no-connect marks 14 -> 0
Other:
- moved on the sheet: J3, LD1
