File: boards/macro system v2 pcb/controller test board.kicad_sch (KiCad schematic)
At the start: 37 parts, among them J1 Conn_01x02, J10 Conn_01x03, J12 Conn_01x02, J15 LED conn, J2 Conn_01x03, J4 Conn_01x06, J5 FH19C-10S-0.5SH10, J6 Conn_01x03, J7 Mirror drive, J8 mdrive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

Commit message: create new LD only mount PCB
Parts:
- R1: value 5M -> 5.1M
- TVS2: renamed from D2; value D -> 35v
- TVS3: renamed from D3; value D -> 3.3v
- TVS4: renamed from D4; value D -> 3.3v
- TVS5: renamed from D5; value D -> 3.3v
- TVS6: renamed from D6; value D -> 3.3v
Other:
- sheet ICE40UP5K ports: added none; removed ADC_A/B, ADC_CLK, ADC_D3, ADC_D4, ADC_D5, ADC_D6, ADC_D7, LED_drive, PWM_DAC_1
Changed lines of the file:
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@@
 	(wire
 		(pts
-			(xy 160.02 132.08) (xy 156.21 132.08)
+			(xy 166.37 132.08) (xy 156.21 132.08)
 		)
 		(stroke
@@
 	(wire
 		(pts
-			(xy 158.75 146.05) (xy 158.75 134.62)
+			(xy 165.1 146.05) (xy 165.1 134.62)
 		)
 		(stroke
@@
 	(wire
 		(pts
-			(xy 160.02 143.51) (xy 160.02 132.08)
+			(xy 166.37 143.51) (xy 166.37 132.08)
 		)
 		(stroke
@@
 	(wire
 		(pts
-			(xy 158.75 146.05) (xy 175.26 146.05)
+			(xy 165.1 146.05) (xy 175.26 146.05)
 		)
 		(stroke
@@
 	(wire
 		(pts
-			(xy 158.75 134.62) (xy 152.4 134.62)
+			(xy 165.1 134.62) (xy 152.4 134.62)
 		)
 		(stroke
@@
 	(wire
 		(pts
-			(xy 160.02 143.51) (xy 175.26 143.51)
+			(xy 166.37 143.51) (xy 175.26 143.51)
 		)
 		(stroke
@@
 		(on_board yes)
 		(dnp no)
-		(property "Reference" "D5"
-			(at 160.274 53.34 90)
+		(property "Reference" "TVS5"
+			(at 161.798 53.34 90)
 			(effects
 				(font
@@
 			)
 		)
-		(property "Value" "D"
+		(property "Value" "3.3v"
 			(at 161.798 51.562 90)
 			(effects
@@
 			(project "controller test board"
 				(path "/e63e39d7-6ac0-4ffd-8aa3-1841a4541b55"
-					(reference "D5")
+					(reference "TVS5")
 					(unit 1)
 				)
@@
 			)
 		)
-		(property "Value" "5M"
+		(property "Value" "5.1M"
 			(at 61.976 74.93 0)
 			(effects
@@
 		(on_board yes)
 		(dnp no)
-		(property "Reference" "D3"
-			(at 152.654 142.24 90)
+		(property "Reference" "TVS3"
+			(at 146.558 141.732 90)
 			(effects
 				(font
@@
 			)
 		)
-		(property "Value" "D"
-			(at 153.924 144.018 90)
+		(property "Value" "3.3v"
+			(at 146.812 143.51 90)
 			(effects
 				(font
@@
 			(project "controller test board"
 				(path "/e63e39d7-6ac0-4ffd-8aa3-1841a4541b55"
-					(reference "D3")
+					(reference "TVS3")
 					(unit 1)
 				)
@@
 		(on_board yes)
 		(dnp no)
-		(property "Reference" "D6"
-			(at 240.284 87.63 90)
+		(property "Reference" "TVS6"
+			(at 241.808 87.63 90)
 			(effects
 				(font
@@
 			)
 		)
-		(property "Value" "D"
+		(property "Value" "3.3v"
 			(at 241.808 85.852 90)
 			(effects
@@
 			(project "controller test board"
 				(path "/e63e39d7-6ac0-4ffd-8aa3-1841a4541b55"
-					(reference "D6")
+					(reference "TVS6")
 					(unit 1)
 				)
@@
 		(on_board yes)
 		(dnp no)
-		(property "Reference" "D2"
-			(at 67.564 74.93 90)
+		(property "Reference" "TVS2"
+			(at 68.834 71.374 90)
 			(effects
 				(font
@@
 			)
 		)
-		(property "Value" "D"
-			(at 68.834 76.708 90)
+		(property "Value" "35v"
+			(at 69.088 73.152 90)
 			(effects
 				(font
@@
 			(project "controller test board"
 				(path "/e63e39d7-6ac0-4ffd-8aa3-1841a4541b55"
-					(reference "D2")
+					(reference "TVS2")
 					(unit 1)
 				)
@@
 		(on_board yes)
 		(dnp no)
-		(property "Reference" "D4"
-			(at 156.464 142.24 90)
+		(property "Reference" "TVS4"
+			(at 156.21 142.24 90)
 			(effects
 				(font
@@
 			)
 		)
-		(property "Value" "D"
-			(at 157.734 144.018 90)
+		(property "Value" "3.3v"
+			(at 156.718 144.018 90)
 			(effects
 				(font
@@
 			(project "controller test board"
 				(path "/e63e39d7-6ac0-4ffd-8aa3-1841a4541b55"
-					(reference "D4")
+					(reference "TVS4")
 					(unit 1)
 				)
@@
 			)
 		)
-		(pin "ADC_CLK" input
-			(at 149.86 80.01 0)
-			(effects
-				(font
-					(size 1.27 1.27)
-				)
-				(justify right)
-			)
-		)
 		(pin "UWB_SCK" input
 			(at 149.86 113.03 0)
@@
 			)
 		)
-		(pin "ADC_D5" input
-			(at 149.86 97.79 0)
-			(effects
-				(font
-					(size 1.27 1.27)
-				)
-				(justify right)
-			)
-		)
-		(pin "ADC_D3" input
-			(at 149.86 90.17 0)
-			(effects
-				(font
-					(size 1.27 1.27)
-				)
-				(justify right)
-			)
-		)
 		(pin "ADC_D0" input
 			(at 149.86 82.55 0)
@@
 			)
 		)
-		(pin "ADC_D6" input
-			(at 149.86 100.33 0)
-			(effects
-				(font
-					(size 1.27 1.27)
-				)
-				(justify right)
-			)
-		)
-		(pin "ADC_D4" input
-			(at 149.86 95.25 0)
-			(effects
-				(font
-					(size 1.27 1.27)
-				)
-				(justify right)
-			)
-		)
 		(pin "ADC_D2" input
 			(at 149.86 87.63 0)
@@
 			)
 		)
-		(pin "ADC_D7" input
-			(at 149.86 102.87 0)
-			(effects
-				(font
-					(size 1.27 1.27)
-				)
-				(justify right)
-			)
-		)
-		(pin "PWM_DAC_1" input
-			(at 149.86 73.66 0)
-			(effects
-				(font
-					(size 1.27 1.27)
-				)
-				(justify right)
-			)
-		)
 		(pin "PWM_DAC_2" input
 			(at 149.86 76.2 0)
@@
 			(effects
 				(font
-					(size 1.27 1.27)
-				)
-				(justify right)
-			)
-		)
-		(pin "LED_drive" input
-			(at 149.86 71.12 0)
-			(effects
-				(font
-					(size 1.27 1.27)
-				)
-				(justify right)
-			)
-		)
-		(pin "ADC_A{slash}B" input
-			(at 149.86 92.71 0)
-			(effects
-				(font
